File: Hardware/laser-theremin-audio.sch (KiCad schematic (older format))
At the start: 17 parts, among them J4 Audio Out, J5 Rack2, J6 Conn_01x01, J8 Conn_01x01, J9 Rack1, U6 LM4861

Commit message: Updating design to final
Parts:
- D12: footprint OPL_Discrete_Semiconductor:SOD-123 -> lib_fp:SOD-123
Changed lines of the file:
@@
 F 0 "D12" H 8705 2900 50  0000 C CNN
 F 1 "D_Schottky" H 8715 3120 50  0001 C CNN
-F 2 "OPL_Discrete_Semiconductor:SOD-123" H 8715 2995 50  0001 C CNN
+F 2 "lib_fp:SOD-123" H 8715 2995 50  0001 C CNN
 F 3 "~" H 8715 2995 50  0001 C CNN
 	1    8715 2995
