File: Hardware/laser-theremin-led.sch (KiCad schematic (older format))
At the start: 14 parts

Commit message: Updating design to final
Parts:
- D10, D11, D7, D8, D9: footprint OPL_Optoelectronics:LED-0603 -> lib_fp:LED-0603
- D5, D6: footprint OPL_Optoelectronics:LED4-SMD-5050 -> lib_fp:LED4-SMD-5050
Changed lines of the file:
@@
 F 0 "D5" H 3224 3721 50  0000 L CNN
 F 1 "SK6812" H 3224 3630 50  0000 L CNN
-F 2 "OPL_Optoelectronics:LED4-SMD-5050" H 2930 3375 50  0001 L TNN
+F 2 "lib_fp:LED4-SMD-5050" H 2930 3375 50  0001 L TNN
 F 3 "https://cdn-shop.adafruit.com/product-files/1138/SK6812+LED+datasheet+.pdf" H 2980 3300 50  0001 L TNN
 	1    2880 3675
@@
 F 0 "D6" H 4324 3721 50  0000 L CNN
 F 1 "SK6812" H 4324 3630 50  0000 L CNN
-F 2 "OPL_Optoelectronics:LED4-SMD-5050" H 4030 3375 50  0001 L TNN
+F 2 "lib_fp:LED4-SMD-5050" H 4030 3375 50  0001 L TNN
 F 3 "https://cdn-shop.adafruit.com/product-files/1138/SK6812+LED+datasheet+.pdf" H 4080 3300 50  0001 L TNN
 	1    3980 3675
@@
 F 0 "D7" V 5969 3388 50  0000 R CNN
 F 1 "LED" V 5878 3388 50  0000 R CNN
-F 2 "OPL_Optoelectronics:LED-0603" H 5930 3505 50  0001 C CNN
+F 2 "lib_fp:LED-0603" H 5930 3505 50  0001 C CNN
 F 3 "~" H 5930 3505 50  0001 C CNN
 	1    5930 3505
@@
 F 0 "D8" V 6469 3388 50  0000 R CNN
 F 1 "LED" V 6378 3388 50  0000 R CNN
-F 2 "OPL_Optoelectronics:LED-0603" H 6430 3505 50  0001 C CNN
+F 2 "lib_fp:LED-0603" H 6430 3505 50  0001 C CNN
 F 3 "~" H 6430 3505 50  0001 C CNN
 	1    6430 3505
@@
 F 0 "D9" V 6969 3388 50  0000 R CNN
 F 1 "LED" V 6878 3388 50  0000 R CNN
-F 2 "OPL_Optoelectronics:LED-0603" H 6930 3505 50  0001 C CNN
+F 2 "lib_fp:LED-0603" H 6930 3505 50  0001 C CNN
 F 3 "~" H 6930 3505 50  0001 C CNN
 	1    6930 3505
@@
 F 0 "D10" V 7464 3388 50  0000 R CNN
 F 1 "LED" V 7373 3388 50  0000 R CNN
-F 2 "OPL_Optoelectronics:LED-0603" H 7425 3505 50  0001 C CNN
+F 2 "lib_fp:LED-0603" H 7425 3505 50  0001 C CNN
 F 3 "~" H 7425 3505 50  0001 C CNN
 	1    7425 3505
@@
 F 0 "D11" V 7964 3388 50  0000 R CNN
 F 1 "LED" V 7873 3388 50  0000 R CNN
-F 2 "OPL_Optoelectronics:LED-0603" H 7925 3505 50  0001 C CNN
+F 2 "lib_fp:LED-0603" H 7925 3505 50  0001 C CNN
 F 3 "~" H 7925 3505 50  0001 C CNN
 	1    7925 3505
