File: Hardware/laser-theremin.kicad_pcb (KiCad board)
At the start: 2 copper layers, 99.4 x 60.4 mm, 97 parts, among them J1 JTAG, J10 Conn_01x01, J11 Conn_01x01, J12 Conn_01x01, J2 Micro_SD_Card_SPI, J3 USB_B_Micro, J4 Audio Out, J5 Conn_01x01, J6 Conn_01x01, J7 OLED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

Commit message: Adding design files and outputs for proto1 and proto2
Parts:
- added D13: D_Schottky, OPL_Discrete_Semiconductor:SOD-123, B.Cu at (122.4, 76.8)
- added G***: LOGO, lib_fp:dczia-text, B.Cu at (177.5, 65.2)
- added G***: LOGO, lib_fp:dczia-text, F.Cu at (100.5, 97.5)
- added G***: LOGO, lib_fp:credits, B.Cu at (172.2, 105.3)
- added G***: LOGO, lib_fp:seeed_logo, B.Cu at (152.2, 86.6)
- added J13: TagConnect, Tag-Connect:TC2050-NL_SMALL, B.Cu at (101.0, 108.1)
- added R31: 20k, Resistor_SMD:R_0402_1005Metric, B.Cu at (149.9, 93.3)
- C14: value 1uF -> 0.33uF
- C15: value 0.33uF -> 1uF
- J1: footprint Connector_PinHeader_1.27mm:PinHeader_2x05_P1.27mm_Vertical -> lib_fp:PinHeader_2x05_P1.27mm_Vertical_Sneaky
- J12: footprint TestPoint:TestPoint_Pad_2.5x2.5mm -> TestPoint:TestPoint_Pad_1.0x1.0mm
- J5: value Conn_01x01 -> Rack2; footprint TestPoint:TestPoint_Pad_2.5x2.5mm -> Connector_PinHeader_2.54mm:PinHeader_1x04_P2.54mm_Vertical; moved to F.Cu
- J8: value Rack2 -> Conn_01x01; footprint Connector_PinHeader_2.54mm:PinHeader_1x04_P2.54mm_Vertical -> TestPoint:TestPoint_Pad_2.5x2.5mm; moved to B.Cu
- R13, R14: value 20k -> 10k
- U3: footprint lib_fp:RIGADO_BMD-340 -> RIGADO_BMD-340
- moved R14 40.4 mm to (190.2, 106.8), turned to 180 degrees
- moved J8 25.7 mm to (180.8, 97.0), turned to 0 degrees
- moved J5 23.8 mm to (171.9, 121.0), turned to 90 degrees
- moved G*** 13.4 mm to (137.5, 105.5)
- moved R13 9.11 mm to (150.1, 102.0)
- moved R20 6.86 mm to (143.5, 95.7)
- moved J1 5.51 mm to (106.4, 104.9)
- moved J12 5.47 mm to (183.1, 69.4)
- moved R15 5.36 mm to (111.4, 110.5)
- moved R26 5.35 mm to (111.8, 109.0)
- moved C15 3.71 mm to (143.6, 98.2)
- moved C14 3.63 mm to (140.9, 95.7), turned to 0 degrees
- moved J10 3.62 mm to (132.1, 100.5)
- moved J11 3.61 mm to (135.8, 100.5)
- moved C6 2.60 mm to (118.2, 97.8)
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Connections:
- net UART_RX renamed Net-(J11-Pad1)
- net UART_TX renamed Net-(J10-Pad1)
- C11 pad 1: GND -> Net-(C11-Pad1)
- C11 pad 2: Net-(C11-Pad2) -> GND
- C14 pad 1: Net-(C14-Pad1) -> Net-(C11-Pad1)
- C14 pad 2: GND -> Net-(C14-Pad2)
- C15 pad 1: Net-(C11-Pad2) -> GND
- D2 pad 1: Net-(C13-Pad1) -> Net-(C12-Pad2)
- D2 pad 2: Net-(C12-Pad2) -> Net-(C13-Pad1)
- J1 pad 10: (no net) -> nRESET
- J1 pad 6: (no net) -> SW0
- J3 pad 2: Net-(C13-Pad1) -> Net-(C12-Pad2)
- J3 pad 3: Net-(C12-Pad2) -> Net-(C13-Pad1)
- J4 pad 2: Net-(J4-Pad2) -> GND
- J4 pad 3: (no net) -> Net-(C14-Pad2)
- J4 pad 4: Net-(J4-Pad4) -> Net-(C14-Pad2)
- J4 pad 6: A+ -> HP_DETECT
- J4 pad 8: A- -> (no net)
- J5 pad 1: Net-(J4-Pad4) -> A-
- J6 pad 1: Net-(J4-Pad2) -> A+
- R12 pad 1: Net-(C11-Pad2) -> Net-(C11-Pad1)
- R13 pad 1: Net-(C15-Pad2) -> AUDIO_SHTDN
- R13 pad 2: Net-(R13-Pad2) -> +3V3
- R14 pad 1: AUDIO_SHUTDOWN -> HP_DETECT
- R20 pad 1: Net-(R13-Pad2) -> Net-(C14-Pad2)
- R20 pad 2: A- -> Net-(R20-Pad2)
- U3 pad 10: S2_2 -> S2_1
- U3 pad 31: (no net) -> HP_DETECT
- U3 pad 32: (no net) -> LED_A
- U3 pad 33: LED_A -> KEY_A
- U3 pad 34: KEY_A -> LED_I
- U3 pad 35: LED_I -> KEY_I
- U3 pad 36: KEY_I -> LED_Z
- U3 pad 37: LED_Z -> KEY_Z
- U3 pad 38: KEY_Z -> LED_C
- U3 pad 39: LED_C -> nRESET
- U3 pad 56: GATE -> SW0
- U3 pad 57: CV -> GATE
- U3 pad 58: (no net) -> CV
- U3 pad 63: AUDIO_SHUTDOWN -> AUDIO_SHTDN
- U3 pad 9: S2_1 -> S2_2
- U6 pad 1: AUDIO_SHUTDOWN -> AUDIO_SHTDN
- U6 pad 2: Net-(C14-Pad1) -> Net-(C15-Pad2)
- U6 pad 3: Net-(C14-Pad1) -> Net-(C15-Pad2)
- U6 pad 4: Net-(R13-Pad2) -> Net-(R20-Pad2)
Routing:
- net HP_DETECT: track 0.00 -> 84.5 mm
- net Net-(C14-Pad2): track 0.00 -> 67.0 mm, vias 0 -> 2
- net Net-(D13-Pad1): track 0.00 -> 60.0 mm, vias 0 -> 4
- net GND: track 212.0 -> 263.2 mm, vias 42 -> 56
- net AUDIO_SHUTDOWN: track 41.2 -> 0.00 mm
- net AUDIO_SHTDN: track 0.00 -> 39.0 mm
- net SW0: track 0.00 -> 21.9 mm, vias 0 -> 3
- net nRESET: track 0.00 -> 21.0 mm, vias 0 -> 1
- net Net-(J4-Pad2): track 14.6 -> 0.00 mm
- net +3V3: track 391.7 -> 404.2 mm, vias 20 -> 23
- net Net-(J10-Pad1): track 40.2 -> 29.0 mm
- net SWDIO: track 9.26 -> 20.0 mm
- net Net-(J4-Pad4): track 10.2 -> 0.00 mm, vias 2 -> 0
- net Net-(R20-Pad2): track 0.00 -> 7.45 mm
- net Net-(R13-Pad2): track 7.45 -> 0.00 mm
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Other:
- board text removed: "@dczia505 @lithochasm luna syntax"
- board text removed: "@hamster"
- board text removed: "DOUT"

Commit message: Updating design to final
Parts:
- added J14: Conn_01x01, TestPoint:TestPoint_Pad_2.5x2.5mm, B.Cu at (158.9, 92.8)
- added J15: Conn_01x01, TestPoint:TestPoint_Pad_2.5x2.5mm, B.Cu at (158.9, 89.1)
- added J16: Conn_01x01, TestPoint:TestPoint_Pad_2.5x2.5mm, B.Cu at (158.9, 84.5)
- D1, D12, D13: footprint OPL_Discrete_Semiconductor:SOD-123 -> lib_fp:SOD-123
- D10, D11, D7, D8, D9: footprint OPL_Optoelectronics:LED-0603 -> lib_fp:LED-0603
- D3, D4: footprint Diode_SMD:D_SOD-323 -> Diode_SMD:D_SOD-323_HandSoldering
- D5, D6: footprint OPL_Optoelectronics:LED4-SMD-5050 -> lib_fp:LED4-SMD-5050
- moved G*** 6.25 mm to (146.0, 86.8)
- moved D3 0.40 mm to (104.8, 89.8)
- moved R29 0.39 mm to (163.7, 109.2)
- turned D1 to 180 degrees
- turned D10 to 0 degrees
- turned D11 to 0 degrees
- turned D12 to 90 degrees
- turned D13 to 180 degrees
- turned D7 to 0 degrees
- turned D8 to 0 degrees
- turned D9 to 0 degrees
Connections:
- SW1 pad 1: (no net) -> RACK_PWR
- SW1 pad 3: RACK_PWR -> (no net)
- U4 pad 1: Net-(D3-Pad2) -> (no net)
- U4 pad 4: (no net) -> Net-(D3-Pad2)
- U5 pad 1: Net-(D4-Pad2) -> (no net)
- U5 pad 4: (no net) -> Net-(D4-Pad2)
Routing:
- net +2V8: track 122.6 -> 133.3 mm, vias 5 -> 7
- net RACK_PWR: track 117.6 -> 125.3 mm, vias 2 -> 4
- net GND: track 263.2 -> 266.7 mm, vias 56 -> 52
- net Net-(D4-Pad2): track 3.86 -> 7.35 mm
- net Net-(D3-Pad2): track 4.68 -> 6.79 mm
- net +3V3: track 404.2 -> 406.3 mm, vias 23 -> 24
- net A-: track 62.8 -> 64.6 mm
- net SCL_2_8: track 99.1 -> 100.6 mm
- net A+: track 62.9 -> 64.3 mm
- net Net-(J10-Pad1): track 29.0 -> 29.8 mm
- net SDA_2_8: track 106.7 -> 107.6 mm
Other:
- board text added: "2.8V"
- board text added: "3.3V"
- board text added: "Assembly Instructions"
- board text added: "BEEP"
- board text added: "GND"
- board text added: "GP1 SDA VCC GP2 SCL GND"
- board text added: "Note: Solder Battery Box First"
- board text added: "SLEEP"
- board text added: "https://bit.ly/2KYaf7k"
