File: Hardware/laser-theremin.sch (KiCad schematic (older format))
At the start: 79 parts, among them J1 JTAG, J10 Conn_01x01, J11 Conn_01x01, J12 Conn_01x01, J2 Micro_SD_Card_SPI, J3 USB_B_Micro, J4 Audio Out, J5 Conn_01x01, J6 Conn_01x01, J7 OLED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

Commit message: Adding design files and outputs for proto1 and proto2
Parts:
- removed C11: 10nF, Capacitor_SMD:C_0402_1005Metric, symbol Device:C_Small
- removed C14: 1uF, Capacitor_SMD:C_0402_1005Metric, symbol Device:C_Small
- removed C15: 0.33uF, Capacitor_SMD:C_0402_1005Metric, symbol Device:C_Small
- removed C16: 0.1uF, Capacitor_SMD:C_0402_1005Metric, symbol Device:C_Small
- removed D12: D_Schottky, OPL_Discrete_Semiconductor:SOD-123, symbol Device:D_Schottky
- removed J4: Audio Out, OPL_Connector:AUDIO8P-SMD-3.5-14.5X6X5MM, symbol OPL_Connector:AUDIO-JACK-SMD-8P_PJ-3536-L6S_
- removed J5, J6: Conn_01x01, TestPoint:TestPoint_Pad_2.5x2.5mm, symbol Connector_Generic:Conn_01x01
- removed J8: Rack2, Connector_PinHeader_2.54mm:PinHeader_1x04_P2.54mm_Vertical, symbol Connector_Generic:Conn_01x04
- removed J9: Rack1, Connector_PinHeader_2.54mm:PinHeader_1x04_P2.54mm_Vertical, symbol Connector_Generic:Conn_01x04
- removed LS1: Speaker, lib_fp:Speaker, symbol Device:Speaker
- removed R12: 1k, Resistor_SMD:R_0402_1005Metric, symbol Device:R
- removed R13, R14, R20: 20k, Resistor_SMD:R_0402_1005Metric, symbol Device:R
- removed U6: LM4861, Package_SO:SOIC-8_3.9x4.9mm_P1.27mm, symbol DCZia_audio_amp:Amplifier_Audio_LM4861
- added D13: D_Schottky, OPL_Discrete_Semiconductor:SOD-123, symbol Device:D_Schottky
- added J13: TagConnect, Tag-Connect:TC2050-NL_SMALL, symbol Connector_Generic:Conn_02x05_Odd_Even
- J1: footprint Connector_PinHeader_1.27mm:PinHeader_2x05_P1.27mm_Vertical -> lib_fp:PinHeader_2x05_P1.27mm_Vertical_Sneaky
- J12: footprint TestPoint:TestPoint_Pad_2.5x2.5mm -> TestPoint:TestPoint_Pad_1.0x1.0mm
- J3: symbol Connector_Specialized:USB_B_Micro -> usb_b_micro:USB_B_Micro
- U3: footprint lib_fp:RIGADO_BMD-340 -> RIGADO_BMD-340
Connections:
- net +3V3: now also J13.1 (Pin_1)
- net +BATT: now also D13.2 (A)
- net CV: now also U3.58 (P1.02); no longer U3.57 (P1.01)
- net GATE: now also U3.57 (P1.01); no longer U3.56 (TRACEDATA[0]/SW0/P1.00)
- net GND: now also J13.3 (Pin_3)
- net KEY_A: now also U3.33 (P0.15/TRACEDATA[2]); no longer U3.34 (P0.16/TRACEDATA[1])
- net KEY_I: now also U3.35 (P0.17); no longer U3.36 (P0.21)
- net KEY_Z: now also U3.37 (P0.19); no longer U3.38 (P0.20)
- net LED_A: now also U3.32 (P0.14); no longer U3.33 (P0.15/TRACEDATA[2])
- net LED_C: now also U3.38 (P0.20); no longer U3.39 (P0.18)
- net LED_I: now also U3.34 (P0.16/TRACEDATA[1]); no longer U3.35 (P0.17)
- net LED_Z: now also U3.36 (P0.21); no longer U3.37 (P0.19)
- net S2_1: now also U3.10 (P0.29); no longer U3.9 (P0.28)
- net S2_2: now also U3.9 (P0.28); no longer U3.10 (P0.29)
- net SWCLK: now also J13.4 (Pin_4)
- net SWDIO: now also J13.2 (Pin_2)
- net HP_DETECT: now reaches U3.31 (P0.13)
- net at C12.2, R10.1: now also D2.1 (K), J3.2 (D-); no longer D2.2 (K), J3.3 (D+)
- net at C13.1, R11.1: now also D2.2 (K), J3.3 (D+); no longer D2.1 (K), J3.2 (D-)
- net nRESET: now reaches J1.10 (Pin_10)
- net nRESET: now also U3.39 (P0.18), J13.10 (Pin_10)
- net SW0: now reaches J1.6 (Pin_6)
- net SW0: now also U3.56 (TRACEDATA[0]/SW0/P1.00), J13.6 (Pin_6)
- net AUDIO_SHUTDOWN renamed AUDIO_SHTDN
- net UART_RX: no longer names the net of J11.1 (Pin_1), U3.24 (P0.08)
- net UART_TX: no longer names the net of J10.1 (Pin_1), U3.22 (P0.06)
- new net: D13.1 (K), J13.7 (Pin_7)
- no-connect marks 30 -> 24
Other:
- note added: "DOUT"
- note added: "RX"
- note added: "TX"
- note removed: "Eurorack Expansion"
- note removed: "mediumrehr Audio"
- moved on the sheet: J1, J10, J11, J12, R21, R22, R25, SW7

Commit message: Updating design to final
Parts:
- added J14, J15, J16: Conn_01x01, TestPoint:TestPoint_Pad_2.5x2.5mm, symbol Connector_Generic:Conn_01x01
- D1, D13: footprint OPL_Discrete_Semiconductor:SOD-123 -> lib_fp:SOD-123
- D3, D4: footprint Diode_SMD:D_SOD-323 -> Diode_SMD:D_SOD-323_HandSoldering
Connections:
- net +2V8: now also J15.1 (Pin_1)
- net +3V3: now also J14.1 (Pin_1)
- net GND: now also J16.1 (Pin_1)
- net RACK_PWR: now also SW1.1 (A); no longer SW1.3 (C)
- net at D4.2 (A), R9.1: now also U5.4 (GPIO0); no longer U5.1 (GPIO1)
- net at D3.2 (A), R8.1: now also U4.4 (GPIO0); no longer U4.1 (GPIO1)
Other:
- moved on the sheet: D3, D4, R8, R9
Changed lines of the file:
@@
 F 0 "D1" H 905 1560 50  0000 C CNN
 F 1 "D_Schottky" H 905 1585 50  0001 C CNN
-F 2 "OPL_Discrete_Semiconductor:SOD-123" H 905 1460 50  0001 C CNN
+F 2 "lib_fp:SOD-123" H 905 1460 50  0001 C CNN
 F 3 "~" H 905 1460 50  0001 C CNN
 	1    905  1460
@@
 F 3 "~" H 1560 1360 50  0001 C CNN
 	1    1560 1360
-	-1   0    0    -1
+	-1   0    0    1
 $EndComp
 $Comp
@@
 L Device:R R9
 U 1 1 5D04B0C2
-P 8565 4675
-F 0 "R9" V 8485 4675 50  0000 C CNN
-F 1 "47k" V 8565 4680 50  0000 C CNN
-F 2 "Resistor_SMD:R_0402_1005Metric" V 8495 4675 50  0001 C CNN
-F 3 "~" H 8565 4675 50  0001 C CNN
-	1    8565 4675
+P 8515 4775
+F 0 "R9" V 8435 4775 50  0000 C CNN
+F 1 "47k" V 8515 4780 50  0000 C CNN
+F 2 "Resistor_SMD:R_0402_1005Metric" V 8445 4775 50  0001 C CNN
+F 3 "~" H 8515 4775 50  0001 C CNN
+	1    8515 4775
 	-1   0    0    1
 $EndComp
@@
 L Device:D_Small D4
 U 1 1 5D04BF2A
-P 8265 4825
-F 0 "D4" H 8265 4980 50  0000 C CNN
-F 1 "1N4148" H 8265 4905 50  0000 C CNN
-F 2 "Diode_SMD:D_SOD-323" V 8265 4825 50  0001 C CNN
-F 3 "~" V 8265 4825 50  0001 C CNN
-	1    8265 4825
-	1    0    0    -1
-$EndComp
-Text GLabel 8125 4825 0    50   Input ~ 0
+P 8270 4925
+F 0 "D4" H 8270 5080 50  0000 C CNN
+F 1 "1N4148" H 8270 5005 50  0000 C CNN
+F 2 "Diode_SMD:D_SOD-323_HandSoldering" V 8270 4925 50  0001 C CNN
+F 3 "~" V 8270 4925 50  0001 C CNN
+	1    8270 4925
+	1    0    0    -1
+$EndComp
+Text GLabel 8130 4925 0    50   Input ~ 0
 TOF1_SHDN
 Wire Wire Line
-	8125 4825 8165 4825
-Wire Wire Line
-	8565 4825 8665 4825
-Wire Wire Line
-	8565 4825 8365 4825
-Connection ~ 8565 4825
+	8130 4925 8170 4925
+Wire Wire Line
+	8515 4925 8370 4925
 $Comp
 L power:+2V8 #PWR0112
 U 1 1 5D0C7D13
-P 8565 4525
-F 0 "#PWR0112" H 8565 4375 50  0001 C CNN
-F 1 "+2V8" H 8580 4698 50  0000 C CNN
-F 2 "" H 8565 4525 50  0001 C CNN
-F 3 "" H 8565 4525 50  0001 C CNN
-	1    8565 4525
+P 8515 4625
+F 0 "#PWR0112" H 8515 4475 50  0001 C CNN
+F 1 "+2V8" H 8530 4798 50  0000 C CNN
+F 2 "" H 8515 4625 50  0001 C CNN
+F 3 "" H 8515 4625 50  0001 C CNN
+	1    8515 4625
 	1    0    0    -1
 $EndComp
@@
 L Device:R R8
 U 1 1 5D0FDBB2
-P 8560 5810
-F 0 "R8" V 8480 5810 50  0000 C CNN
-F 1 "47k" V 8560 5815 50  0000 C CNN
-F 2 "Resistor_SMD:R_0402_1005Metric" V 8490 5810 50  0001 C CNN
-F 3 "~" H 8560 5810 50  0001 C CNN
-	1    8560 5810
+P 8515 5910
+F 0 "R8" V 8435 5910 50  0000 C CNN
+F 1 "47k" V 8515 5915 50  0000 C CNN
+F 2 "Resistor_SMD:R_0402_1005Metric" V 8445 5910 50  0001 C CNN
+F 3 "~" H 8515 5910 50  0001 C CNN
+	1    8515 5910
 	-1   0    0    1
 $EndComp
@@
 L Device:D_Small D3
 U 1 1 5D0FDBBC
-P 8260 5960
-F 0 "D3" H 8260 6115 50  0000 C CNN
-F 1 "1N4148" H 8260 6040 50  0000 C CNN
-F 2 "Diode_SMD:D_SOD-323" V 8260 5960 50  0001 C CNN
-F 3 "~" V 8260 5960 50  0001 C CNN
-	1    8260 5960
-	1    0    0    -1
-$EndComp
-Text GLabel 8120 5960 0    50   Input ~ 0
+P 8260 6060
+F 0 "D3" H 8260 6215 50  0000 C CNN
+F 1 "1N4148" H 8260 6140 50  0000 C CNN
+F 2 "Diode_SMD:D_SOD-323_HandSoldering" V 8260 6060 50  0001 C CNN
+F 3 "~" V 8260 6060 50  0001 C CNN
+	1    8260 6060
+	1    0    0    -1
+$EndComp
+Text GLabel 8120 6060 0    50   Input ~ 0
 TOF2_SHDN
 Wire Wire Line
-	8120 5960 8160 5960
-Wire Wire Line
-	8560 5960 8660 5960
-Wire Wire Line
-	8560 5960 8360 5960
-Connection ~ 8560 5960
+	8120 6060 8160 6060
+Wire Wire Line
+	8515 6060 8660 6060
+Wire Wire Line
+	8515 6060 8360 6060
+Connection ~ 8515 6060
 $Comp
 L power:+2V8 #PWR0115
 U 1 1 5D0FDBCB
-P 8560 5660
-F 0 "#PWR0115" H 8560 5510 50  0001 C CNN
-F 1 "+2V8" H 8575 5833 50  0000 C CNN
-F 2 "" H 8560 5660 50  0001 C CNN
-F 3 "" H 8560 5660 50  0001 C CNN
-	1    8560 5660
+P 8515 5760
+F 0 "#PWR0115" H 8515 5610 50  0001 C CNN
+F 1 "+2V8" H 8530 5933 50  0000 C CNN
+F 2 "" H 8515 5760 50  0001 C CNN
+F 3 "" H 8515 5760 50  0001 C CNN
+	1    8515 5760
 	1    0    0    -1
 $EndComp
@@
 NoConn ~ 1310 3515
 NoConn ~ 1310 3615
-NoConn ~ 8660 6060
-NoConn ~ 8665 4925
+NoConn ~ 8660 5960
+NoConn ~ 8665 4825
 NoConn ~ 7375 3105
 NoConn ~ 1360 1260
@@
 F 0 "D13" H 1155 4120 50  0000 C CNN
 F 1 "D_Schottky" H 1160 4345 50  0001 C CNN
-F 2 "OPL_Discrete_Semiconductor:SOD-123" H 1160 4220 50  0001 C CNN
+F 2 "lib_fp:SOD-123" H 1160 4220 50  0001 C CNN
 F 3 "~" H 1160 4220 50  0001 C CNN
 	1    1160 4220
@@
 	0    -1   -1   0
 $EndComp
+Wire Wire Line
+	8665 4925 8515 4925
+Connection ~ 8515 4925
+$Comp
+L Connector_Generic:Conn_01x01 J14
+U 1 1 5D0D3AC0
+P 6360 5910
+F 0 "J14" H 6555 5880 50  0000 R CNN
+F 1 "Conn_01x01" V 6233 5822 50  0001 R CNN
+F 2 "TestPoint:TestPoint_Pad_2.5x2.5mm" H 6360 5910 50  0001 C CNN
+F 3 "~" H 6360 5910 50  0001 C CNN
+	1    6360 5910
+	-1   0    0    1
+$EndComp
+$Comp
+L Connector_Generic:Conn_01x01 J15
+U 1 1 5D0D4AE2
+P 6360 6110
+F 0 "J15" H 6555 6080 50  0000 R CNN
+F 1 "Conn_01x01" V 6233 6022 50  0001 R CNN
+F 2 "TestPoint:TestPoint_Pad_2.5x2.5mm" H 6360 6110 50  0001 C CNN
+F 3 "~" H 6360 6110 50  0001 C CNN
+	1    6360 6110
+	-1   0    0    1
+$EndComp
+$Comp
+L Connector_Generic:Conn_01x01 J16
+U 1 1 5D0D4D6A
+P 6360 6310
+F 0 "J16" H 6555 6280 50  0000 R CNN
+F 1 "Conn_01x01" V 6233 6222 50  0001 R CNN
+F 2 "TestPoint:TestPoint_Pad_2.5x2.5mm" H 6360 6310 50  0001 C CNN
+F 3 "~" H 6360 6310 50  0001 C CNN
+	1    6360 6310
+	-1   0    0    1
+$EndComp
+$Comp
+L power:GND #PWR014
+U 1 1 5D0D5718
+P 6560 6310
+F 0 "#PWR014" H 6560 6060 50  0001 C CNN
+F 1 "GND" H 6560 6170 50  0000 C CNN
+F 2 "" H 6560 6310 50  0001 C CNN
+F 3 "" H 6560 6310 50  0001 C CNN
+	1    6560 6310
+	1    0    0    -1
+$EndComp
+$Comp
+L power:+2V8 #PWR012
+U 1 1 5D0D5C56
+P 6560 6110
+F 0 "#PWR012" H 6560 5960 50  0001 C CNN
+F 1 "+2V8" V 6555 6335 50  0000 C CNN
+F 2 "" H 6560 6110 50  0001 C CNN
+F 3 "" H 6560 6110 50  0001 C CNN
+	1    6560 6110
+	0    1    1    0
+$EndComp
+$Comp
+L power:+3V3 #PWR05
+U 1 1 5D0D6CCF
+P 6560 5910
+F 0 "#PWR05" H 6560 5760 50  0001 C CNN
+F 1 "+3V3" V 6555 6135 50  0000 C CNN
+F 2 "" H 6560 5910 50  0001 C CNN
+F 3 "" H 6560 5910 50  0001 C CNN
+	1    6560 5910
+	0    1    1    0
+$EndComp
 $EndSCHEMATC
